Commit message: new pc

File: controller/urdf/panda.urdf (robot description, URDF)
Before this commit: robot panda, 12 links, 11 joints
Links:
- removed link panda_leftfinger
- removed link panda_rightfinger
Joints:
- removed joint panda_finger_joint1
- removed joint panda_finger_joint2

Commit message: t

File: controller/urdf/panda.urdf (robot description, URDF)
Before this commit: robot panda, 10 links, 9 joints
Joints:
- joint panda_hand_joint: origin xyz=0 0 0 rpy=0 0 -0.785398163397 -> xyz=0 0 0.1 rpy=0 0 -0.785398163397
